File: PSB(LPF Design)/PSB (LPF Design).kicad_pcb (KiCad board)
At the start: 2 copper layers, 75.8 x 44.5 mm, 21 parts

Commit message: .
Parts:
- added G***: LOGO, logo?:BME_LOGO, F.Cu at (129.0, 126.5)
- added G***: LOGO, logo?:lena, F.Cu at (162.5, 97.5)

Commit message: .
Parts:
- removed the G*** at (162.5, 97.5)
Other:
- board text added: "In"
- board text added: "Out"
- board text added: "V+"
- board text added: "V-"
